File: X15-ESC-CONTROLLER - Copy.brd (EAGLE design)
At the start: 51.6 x 34.2 mm, 27 parts, among them IC1 OP-AMP, J1 3V3 -SWCLK-GND-SWDIO- NRST, Y1 ECS-80-S-4X

Commit message: Almost Finished Rewiring
Look at the copy
Parts:
- moved U$3 45.0 mm to (46.5, 11.8), turned to 180 degrees
- moved J3 42.6 mm to (9.96, 24.5), turned to 0 degrees
- moved Y1 38.7 mm to (2.67, 28.1), turned to 90 degrees
- moved C8 35.4 mm to (1.65, 20.9), turned to 270 degrees
- moved R1 33.5 mm to (9.19, 16.6), turned to 180 degrees
- moved U$4 29.5 mm to (22.7, 29.2), turned to 270 degrees
- moved C1 28.4 mm to (2.46, 18.7), turned to 180 degrees
- moved C3 26.7 mm to (3.51, 1.75), turned to 180 degrees
- moved C6 26.4 mm to (6.88, 27.3)
- moved D1 23.3 mm to (2.79, 14.7), turned to 0 degrees
- moved U$6 21.6 mm to (24.8, 5.21), turned to 90 degrees
- moved R4 19.4 mm to (9.45, 19.7), turned to 0 degrees
- moved C7 19.3 mm to (4.19, 21.4), turned to 0 degrees
- moved C5 19.2 mm to (6.93, 29.4), turned to 180 degrees
- moved R5 19.0 mm to (6.38, 20.5), turned to 270 degrees
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Routing:
- net N$3: track 7.91 -> 52.9 mm, vias 0 -> 4
- net GND: track 125.0 -> 157.0 mm, vias 9 -> 10
- net TIM3_CH2: track 3.07 -> 33.3 mm, vias 0 -> 2
- net TIM3_CH4: track 4.12 -> 31.5 mm, vias 0 -> 4
- net N$2: track 7.91 -> 35.0 mm
- net ADC_IN1: track 4.48 -> 30.7 mm, vias 0 -> 1
- net TLM_2: track 7.56 -> 33.0 mm, vias 0 -> 2
- net TIM3_CH3: track 3.59 -> 28.9 mm, vias 0 -> 4
- net SWCLK: track 0.00 -> 24.7 mm
- net SWDIO: track 0.00 -> 23.7 mm, vias 0 -> 2
- net +3V3: track 73.8 -> 95.0 mm, vias 4 -> 8
- net NRST: track 31.9 -> 11.2 mm, vias 1 -> 0
- net TIM2_CH1: track 10.8 -> 27.0 mm
- net TIM2_CH4: track 36.9 -> 20.9 mm
- net CAN_RX: track 0.00 -> 15.2 mm, vias 0 -> 2
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